Commit message: refactor(diff-drive): Apply suggestions from code review
- Refactored the update() method. Removed unneccessary data structures.
- Make the CI work.

File: diff_drive_controller/test/config/sphere_wheel.xacro (robot description, xacro)
@@ -11,5 +11,5 @@
         <origin xyz="0 0 0" rpy="0 0 0"/>
         <geometry>
-          <sphere radius="${wheel_radius}"/>
+          <sphere radius="${radius}"/>
         </geometry>
       </visual>
@@ -17,5 +17,5 @@
         <origin xyz="0 0 0" rpy="0 0 0"/>
         <geometry>
-          <sphere radius="${wheel_radius}"/>
+          <sphere radius="${radius}"/>
         </geometry>
       </collision>

File: diff_drive_controller/test/config/square_wheel.xacro (robot description, xacro)
@@ -12,5 +12,5 @@
         <geometry>
           <!-- use boxes for wheels, scale radius to account for "circumference" difference -->
-          <box size="${wheel_radius*1.11} ${wheel_radius*1.11} ${wheel_radius*1.11} "/>
+          <box size="${radius*1.11} ${radius*1.11} ${radius*1.11} "/>
         </geometry>
       </visual>
@@ -18,5 +18,5 @@
         <origin xyz="0 0 0" rpy="0 0 0"/>
         <geometry>
-          <box size="${wheel_radius*1.11} ${wheel_radius*1.11} ${wheel_radius*1.11} "/>
+          <box size="${radius*1.11} ${radius*1.11} ${radius*1.11} "/>
         </geometry>
       </collision>

File: diff_drive_controller/test/config/wheel.xacro (robot description, xacro)
@@ -11,5 +11,5 @@
         <origin xyz="0 0 0" rpy="0 0 0"/>
         <geometry>
-          <cylinder radius="${wheel_radius}" length="${thickness}"/>
+          <cylinder radius="${radius}" length="${thickness}"/>
         </geometry>
       </visual>
@@ -17,5 +17,5 @@
         <origin xyz="0 0 0" rpy="0 0 0"/>
         <geometry>
-          <cylinder radius="${wheel_radius}" length="${thickness}"/>
+          <cylinder radius="${radius}" length="${thickness}"/>
         </geometry>
       </collision>
